File: Hardware/Control_PCB/KiCAD_Project/control_pcb/control_pcb.kicad_pcb (KiCad board)
At the start: 4 copper layers, 82.6 x 76.2 mm, 112 parts, among them J1 Conn_01x02, J2 ISP, J3 Spare, J4 XBee ISP, J5 XBee_uC_ISP, J6 Micro_SD_Card_Det, J7 SD_uC_ISP, J8 External Switch, J9 Battery, Q1 BSS138, SW1 ID Select, U1 STM32F103CBT6, U2 XTend, U3 ATmega328P-AU, U4 ATmega328P-AU, U5 IF-D96F, U6 TC4S584F, U7 MAX-M8C, U8 SPX3819M5-L-3-3, U9 1-0000946, Y1 8MHz, Y2 8MHz, Y3 8MHz

Commit message: R42: 1-460 -> 1-678
Parts:
- R42: value 10 -> 1-0000678
Connections:
- J4 pad 5: (no net) -> Net-(J4-Pad5)
- J4 pad 7: (no net) -> Net-(J4-Pad7)
- U1 pad 1: (no net) -> Net-(U1-Pad1)
- U1 pad 10: (no net) -> Net-(U1-Pad10)
- U1 pad 11: (no net) -> Net-(U1-Pad11)
- U1 pad 12: (no net) -> /Unused_Fiber_Ser_TX
- U1 pad 14: (no net) -> Net-(U1-Pad14)
- U1 pad 17: (no net) -> Net-(U1-Pad17)
- U1 pad 2: (no net) -> Net-(U1-Pad2)
- U1 pad 20: (no net) -> Net-(U1-Pad20)
- U1 pad 25: (no net) -> Net-(U1-Pad25)
- U1 pad 26: (no net) -> Net-(U1-Pad26)
- U1 pad 27: (no net) -> Net-(U1-Pad27)
- U1 pad 28: (no net) -> Net-(U1-Pad28)
- U1 pad 29: (no net) -> Net-(U1-Pad29)
- U1 pad 3: (no net) -> Net-(U1-Pad3)
- U1 pad 32: (no net) -> Net-(U1-Pad32)
- U1 pad 38: (no net) -> Net-(U1-Pad38)
- U1 pad 4: (no net) -> Net-(U1-Pad4)
- U1 pad 43: (no net) -> Net-(U1-Pad43)
- U1 pad 45: (no net) -> Net-(U1-Pad45)
- U1 pad 46: (no net) -> Net-(U1-Pad46)
- U2 pad 12: (no net) -> Net-(U2-Pad12)
- U2 pad 14: (no net) -> Net-(U2-Pad14)
- U2 pad 15: (no net) -> Net-(U2-Pad15)
- U2 pad 16: (no net) -> Net-(U2-Pad16)
- U2 pad 17: (no net) -> Net-(U2-Pad17)
- U2 pad 18: (no net) -> Net-(U2-Pad18)
- U2 pad 19: (no net) -> Net-(U2-Pad19)
- U2 pad 20: (no net) -> Net-(U2-Pad20)
- U2 pad 21: (no net) -> Net-(U2-Pad21)
- U2 pad 23: (no net) -> Net-(U2-Pad23)
- U2 pad 24: (no net) -> Net-(U2-Pad24)
- U2 pad 25: (no net) -> Net-(U2-Pad25)
- U2 pad 26: (no net) -> Net-(U2-Pad26)
- U2 pad 27: (no net) -> Net-(U2-Pad27)
- U2 pad 28: (no net) -> Net-(U2-Pad28)
- U2 pad 30: (no net) -> Net-(U2-Pad30)
- U2 pad 31: (no net) -> Net-(U2-Pad31)
- U2 pad 32: (no net) -> Net-(U2-Pad32)
- U2 pad 33: (no net) -> Net-(U2-Pad33)
- U2 pad 34: (no net) -> Net-(U2-Pad34)
- U2 pad 36: (no net) -> Net-(U2-Pad36)
- U2 pad 37: (no net) -> Net-(U2-Pad37)
- U2 pad 5: (no net) -> Net-(U2-Pad5)
- U2 pad 6: (no net) -> Net-(U2-Pad6)
- U2 pad 7: (no net) -> Net-(U2-Pad7)
- U2 pad 8: (no net) -> Net-(U2-Pad8)
- U2 pad 9: (no net) -> Net-(U2-Pad9)
- U3 pad 11: (no net) -> Net-(U3-Pad11)
- U3 pad 12: (no net) -> Net-(U3-Pad12)
- U3 pad 13: (no net) -> Net-(U3-Pad13)
- U3 pad 14: (no net) -> Net-(U3-Pad14)
- U3 pad 19: (no net) -> Net-(U3-Pad19)
- U3 pad 2: (no net) -> Net-(U3-Pad2)
- U3 pad 22: (no net) -> Net-(U3-Pad22)
- U3 pad 26: (no net) -> Net-(U3-Pad26)
- U3 pad 27: (no net) -> Net-(U3-Pad27)
- U3 pad 28: (no net) -> Net-(U3-Pad28)
- U3 pad 31: (no net) -> Net-(U3-Pad31)
- U4 pad 1: (no net) -> Net-(U4-Pad1)
- U4 pad 10: (no net) -> Net-(U4-Pad10)
- U4 pad 11: (no net) -> Net-(U4-Pad11)
- U4 pad 14: (no net) -> Net-(U4-Pad14)
- U4 pad 19: (no net) -> Net-(U4-Pad19)
- U4 pad 22: (no net) -> Net-(U4-Pad22)
- U4 pad 23: (no net) -> Net-(U4-Pad23)
- U4 pad 24: (no net) -> Net-(U4-Pad24)
- U4 pad 25: (no net) -> Net-(U4-Pad25)
- U4 pad 26: (no net) -> Net-(U4-Pad26)
- U4 pad 27: (no net) -> Net-(U4-Pad27)
- U4 pad 28: (no net) -> Net-(U4-Pad28)
- U4 pad 32: (no net) -> Net-(U4-Pad32)
- U6 pad 1: (no net) -> Net-(U6-Pad1)
- U7 pad 13: (no net) -> Net-(U7-Pad13)
- U7 pad 14: (no net) -> Net-(U7-Pad14)
- U7 pad 15: (no net) -> Net-(U7-Pad15)
- U7 pad 16: (no net) -> Net-(U7-Pad16)
- U7 pad 17: (no net) -> Net-(U7-Pad17)
- U7 pad 18: (no net) -> Net-(U7-Pad18)
- U7 pad 5: (no net) -> Net-(U7-Pad5)
- U7 pad 9: (no net) -> Net-(U7-Pad9)
- U8 pad 4: (no net) -> Net-(U8-Pad4)
- U9 pad 3: (no net) -> Net-(U9-Pad3)
- U9 pad 5: (no net) -> Net-(U9-Pad5)
- U9 pad 8: (no net) -> Net-(U9-Pad8)

Commit message: Update GERBERS to match production
Other:
- net class Default removed
