File: Hardware/Tracker_PCB/KiCAD_Project/tracker/tracker.kicad_pcb (KiCad board)
At the start: 4 copper layers, 78.7 x 57.2 mm, 58 parts, among them J1 RockBlock9603, J2 ICSP, J4 Battery, Q1 BSS138, Q2 BSS138, SW1 SW_SPST, U1 XBee, U2 ATmega328P-AU, U3 TSR2, U4 RockBlockMechanical, U5 ublox_SAM-M8Q, U6 MIC5219-3.3YM5, Y1 16MHz

Commit message: Update GERBERS to match production
Other:
- net class Default removed
