File: PCBs/Motor_Control_PCB/KiCAD_Project/motor_control.kicad_pcb (KiCad board)
At the start: 2 copper layers, 58.4 x 45.7 mm, 53 parts, among them J1 NP_Conn_01x06, J2 NP_Conn_01x02, J3 NP_Conn_01x04, J4 NP_Conn_01x04, J5 NP_Conn_01x04, J6 NP_Conn_01x04, J7 NP_Conn_01x02_Relief, J8 NP_Conn_01x02_Relief, U1 1-0000452, U2 1-0001532, U3 1-0000207, U4 1-0000196, Y1 1-0000721

Commit message: Fixed Motor PCB ERC Issues and Copper to Edge Clearence
Other:
- copper layers 2 -> 4
Changed lines of the file:
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@@
 	(generator_version "8.0")
 	(general
-		(thickness 0.57)
+		(thickness 2.446)
 		(legacy_teardrops no)
 	)
@@
 	(layers
 		(0 "F.Cu" signal)
+		(1 "In1.Cu" signal)
+		(2 "In2.Cu" signal)
 		(31 "B.Cu" signal)
 		(32 "B.Adhes" user "B.Adhesive")
@@
 			(layer "dielectric 1"
 				(type "core")
-				(thickness 0.48)
+				(thickness 0.762)
+				(material "FR4")
+				(epsilon_r 4.5)
+				(loss_tangent 0.02)
+			)
+			(layer "In1.Cu"
+				(type "copper")
+				(thickness 0.035)
+			)
+			(layer "dielectric 2"
+				(type "prepreg")
+				(thickness 0.762)
+				(material "FR4")
+				(epsilon_r 4.5)
+				(loss_tangent 0.02)
+			)
+			(layer "In2.Cu"
+				(type "copper")
+				(thickness 0.035)
+			)
+			(layer "dielectric 3"
+				(type "core")
+				(thickness 0.762)
 				(material "FR4")
 				(epsilon_r 4.5)
@@
 			)
 		)
-		(sheetname "Root")
-		(sheetfile "motor_control.kicad_sch")
-		(attr exclude_from_pos_files)
+		(attr exclude_from_pos_files exclude_from_bom)
 		(fp_circle
 			(center 0 0)
@@
 			)
 		)
-		(sheetname "Root")
-		(sheetfile "motor_control.kicad_sch")
-		(attr exclude_from_pos_files)
+		(attr exclude_from_pos_files exclude_from_bom)
 		(fp_circle
 			(center 0 0)
@@
 			)
 		)
-		(sheetname "Root")
-		(sheetfile "motor_control.kicad_sch")
-		(attr exclude_from_pos_files)
+		(attr exclude_from_pos_files exclude_from_bom)
 		(fp_circle
 			(center 0 0)
@@
 			)
 		)
-		(sheetname "Root")
-		(sheetfile "motor_control.kicad_sch")
-		(attr exclude_from_pos_files)
+		(attr exclude_from_pos_files exclude_from_bom)
 		(fp_circle
 			(center 0 0)
@@
 		)
 		(height 9.09)
-		(gr_text "1500.0000 mils"
+		(gr_text "1.5000 in"
 			(at 176.85 99.06 90)
 			(layer "Dwgs.User")
@@
 		)
 		(height 9.362407)
-		(gr_text "2300.0000 mils"
+		(gr_text "2.3000 in"
 			(at 143.51 69.497594 1.961512481e-06)
 			(layer "Dwgs.User")
@@
 		)
 		(height 10.906184)
-		(gr_text "1800.0000 mils"
+		(gr_text "1.8000 in"
 			(at 106.053816 99.060001 89.99999749)
 			(layer "Dwgs.User")
@@
 		)
 		(height -9.89)
-		(gr_text "2000.0000 mils"
+		(gr_text "2.0000 in"
 			(at 143.51 126.85 0)
 			(layer "Dwgs.User")
